File: romeo-pcb.kicad_pcb (KiCad board)
At the start: 2 copper layers, 247.6 x 99.2 mm, 138 parts, among them J1 AVR-ISP-6, SW0 KEYSW, SW1 KEYSW, SW10 KEYSW, SW11 KEYSW, SW12 KEYSW, SW13 KEYSW, SW14 KEYSW, SW15 KEYSW, SW16 KEYSW, SW17 KEYSW, SW18 KEYSW, SW19 KEYSW, SW2 KEYSW, SW20 KEYSW, SW21 KEYSW, SW22 KEYSW, SW23 KEYSW, SW24 KEYSW, SW25 KEYSW, SW26 KEYSW, SW27 KEYSW, SW28 KEYSW, SW29 KEYSW, SW3 KEYSW, SW30 KEYSW, SW31 KEYSW, SW32 KEYSW, SW33 KEYSW, SW34 KEYSW, SW35 KEYSW, SW36 KEYSW, SW37 KEYSW, SW38 KEYSW, SW39 KEYSW, SW4 KEYSW, SW40 KEYSW, SW41 KEYSW, SW42 KEYSW, SW43 KEYSW, SW44 KEYSW, SW45 KEYSW, SW46 KEYSW, SW47 KEYSW, SW5 KEYSW, SW6 KEYSW, SW7 KEYSW, SW8 KEYSW, SW9 KEYSW, U1 ATmega328P-PU, Y1 Crystal

Commit message: Add new layout to romeo keyboard
Add the new layout (based on CC45) to make the keyboard more convenient to use
Update footprints to match this rev1.2
Parts:
- removed the G*** at (115.0, 136.9) (x2)
- removed the G*** at (176.0, 118.1) (x2)
- removed the G*** at (176.1, 101.8)
- removed the G*** at (27.6, 54.1)
- removed the G*** at (267.3, 54.1)
- removed the G*** at (127.3, 131.5) (x2)
- removed the G*** at (161.8, 133.0)
- removed the G*** at (188.3, 123.5) (x2)
- removed the REF** at (229.3, 123.3)
- removed the REF** at (65.6, 123.3)
- removed the REF** at (50.8, 85.2)
- removed the REF** at (244.2, 85.2)
- removed the REF** at (147.4, 85.2)
- removed the REF** at (267.3, 46.9)
- removed the REF** at (267.3, 61.2)
- removed the REF** at (27.7, 61.2)
- removed the REF** at (27.7, 47.2)
- removed ST39: 6.25U, cftkb:MX-6.25U-Stabilizer
- removed the SW45 at (38.1, 89.7)
- removed the SW46 at (38.1, 108.7)
- added D23: D_Small, cftkb:D_DO-35_SOD27_P5.08mm_Horizontal, F.Cu at (262.4, 53.7)
- added G***: LOGO, logos:TOPY 4MM MASK, F.Cu at (27.7, 54.0)
- added G***: LOGO, logos:TOPY 4MM MASK, F.Cu at (267.3, 54.0)
- added REF**: MountingHole_2.2mm_M2_Pad, cftkb:MountingHole_2.2mm_M2_Pad, F.Cu at (267.4, 46.9)
- added REF**: MountingHole_2.2mm_M2_Pad, cftkb:MountingHole_2.2mm_M2_Pad, F.Cu at (244.2, 85.2)
- added REF**: MountingHole_2.2mm_M2_Pad, cftkb:MountingHole_2.2mm_M2_Pad, F.Cu at (267.4, 61.2)
- added REF**: MountingHole_2.2mm_M2_Pad, cftkb:MountingHole_2.2mm_M2_Pad, F.Cu at (229.4, 123.3)
- added REF**: MountingHole_2.2mm_M2_Pad, cftkb:MountingHole_2.2mm_M2_Pad, F.Cu at (50.8, 85.2)
- added REF**: MountingHole_2.2mm_M2_Pad, cftkb:MountingHole_2.2mm_M2_Pad, F.Cu at (27.7, 47.2)
- added REF**: MountingHole_2.2mm_M2_Pad, cftkb:MountingHole_2.2mm_M2_Pad, F.Cu at (27.7, 61.2)
- added REF**: MountingHole_2.2mm_M2_Pad, cftkb:MountingHole_2.2mm_M2_Pad, F.Cu at (65.7, 123.3)
- added REF**: MountingHole_2.2mm_M2_Pad, cftkb:MountingHole_2.2mm_M2_Pad, F.Cu at (147.5, 85.2)
- added Ref**: Val**, cftkb:rev_num, F.Cu at (189.0, 123.5)
- added Ref**: Val**, cftkb:author_footprint, F.Cu at (188.0, 119.5)
- added Ref**: Val**, cftkb:author_footprint, B.Cu at (97.0, 132.0)
- added Ref**: Val**, cftkb:rev_num, B.Cu at (96.0, 136.0)
- added SW13: KEYSW, cftkb:SW_Cherry_MX1A_2.00u_PCBNOSCREEN, F.Cu at (254.8, 70.6)
- added SW14: KEYSW, cftkb:SW_Cherry_MX1A_1.00u_PCB-NOSCREEN, F.Cu at (231.0, 89.7)
- added SW48: KEYSW, cftkb:SW_Cherry_MX1A_1.25u_PCBNOSCREEN, F.Cu at (219.1, 127.8)
- added SW49: KEYSW, cftkb:SW_Cherry_MX1A_1.00u_PCB-NOSCREEN, F.Cu at (240.5, 127.8)
- added SW50: KEYSW, cftkb:SW_Cherry_MX1A_1.25u_PCBNOSCREEN, F.Cu at (261.9, 127.8)
- added SW51: KEYSW, cftkb:SW_Cherry_MX1A_1.25u_PCBNOSCREEN, F.Cu at (38.1, 127.8)
- added SW52: KEYSW, cftkb:SW_Cherry_MX1A_1.00u_PCB-NOSCREEN, F.Cu at (59.5, 127.8)
- F1: value 100mA -> 500mA
- SW1: renamed from SW0; footprint cftkb:SW_Cherry_MX1A_1.50u_PCBNOSCREEN -> cftkb:SW_Cherry_MX1A_1.00u_PCB-NOSCREEN
- SW12: renamed from SW11; footprint cftkb:SW_Cherry_MX1A_1.50u_PCBNOSCREEN -> cftkb:SW_Cherry_MX1A_1.00u_PCB-NOSCREEN
- SW15: renamed from SW12; footprint cftkb:SW_Cherry_MX1A_1.75u_PCBNOSCREEN -> cftkb:SW_Cherry_MX1A_1.25u_PCBNOSCREEN
- SW25: renamed from SW22; footprint cftkb:SW_Cherry_MX1A_2.25u_PCBNOSCREEN -> cftkb:SW_Cherry_MX1A_1.75u_PCBNOSCREEN
- SW26: renamed from SW23; footprint cftkb:SW_Cherry_MX1A_2.25u_PCBNOSCREEN -> cftkb:SW_Cherry_MX1A_1.75u_PCBNOSCREEN
- SW37: renamed from SW33; footprint cftkb:SW_Cherry_MX1A_1.75u_PCBNOSCREEN -> cftkb:SW_Cherry_MX1A_1.25u_PCBNOSCREEN
- SW38: renamed from SW34; footprint cftkb:SW_Cherry_MX1A_1.25u_PCBNOSCREEN -> cftkb:SW_Cherry_MX1A_1.50u_PCBNOSCREEN
- SW40: renamed from SW36; footprint cftkb:SW_Cherry_MX1A_1.00u_PCB-NOSCREEN -> cftkb:SW_Cherry_MX1A_1.50u_PCBNOSCREEN
- SW42: renamed from SW40; footprint cftkb:SW_Cherry_MX1A_1.00u_PCB-NOSCREEN -> MX_Only:MXOnly-2.75U-ReversedStabilizers-NoLED
- SW43: renamed from SW41; footprint cftkb:SW_Cherry_MX1A_2.75u_PCB_NOSCREEN -> cftkb:SW_Cherry_MX1A_1.50u_PCBNOSCREEN
- SW44: renamed from SW42; footprint cftkb:SW_Cherry_MX1A_1.25u_PCBNOSCREEN -> cftkb:SW_Cherry_MX1A_1.00u_PCB-NOSCREEN
- SW45: renamed from SW43; footprint cftkb:SW_Cherry_MX1A_1.00u_PCB-NOSCREEN -> cftkb:SW_Cherry_MX1A_1.50u_PCBNOSCREEN
- SW46: renamed from SW44; footprint cftkb:SW_Cherry_MX1A_1.25u_PCBNOSCREEN -> cftkb:SW_Cherry_MX1A_1.00u_PCB-NOSCREEN
- SW47: renamed from SW39; footprint cftkb:SW_Cherry_MX1A_1.00u_PCB-NOSCREEN -> MX_Only:MXOnly-6.25U-ReversedStabilizers-NoLED
- SW53: renamed from SW37; footprint cftkb:SW_Cherry_MX1A_1.25u_PCBNOSCREEN -> cftkb:SW_Cherry_MX1A_1.00u_PCB-NOSCREEN
- moved SW46 57.2 mm to (264.3, 70.6)
- moved SW43 31.0 mm to (211.9, 127.8)
- moved G*** 26.2 mm to (188.0, 133.5)
- moved SW42 24.2 mm to (169.0, 132.9)
- moved SW45 19.0 mm to (259.6, 127.8)
- moved SW44 16.7 mm to (235.7, 127.8)
- moved SW12 14.3 mm to (245.3, 70.6)
- moved SW10 9.53 mm to (207.2, 70.6)
- moved SW11 9.53 mm to (226.2, 70.6)
- moved SW16 9.53 mm to (59.5, 89.7)
- moved SW17 9.53 mm to (78.6, 89.7)
- moved SW18 9.53 mm to (97.6, 89.7)
- moved SW2 9.53 mm to (54.8, 70.6)
- moved SW20 9.53 mm to (135.7, 89.7)
- moved SW21 9.53 mm to (154.8, 89.7)
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- renumbered C3 to C1, C4 to C2, C5 to C3, C1 to C4, C2 to C5, D0 to D1, D9 to D10, D10 to D11, D11 to D12, D12 to D13, D13 to D14, D14 to D15, D15 to D16, D16 to D17, D17 to D18, D18 to D19, D1 to D2, D19 to D20, D20 to D21, D21 to D22, D22 to D24, D23 to D25, D47 to D26, D24 to D27, D25 to D28, D26 to D29, D2 to D3, D27 to D30, D28 to D31, D29 to D32, D30 to D33, D31 to D34, D32 to D35, D33 to D36, D34 to D37, D35 to D38, D36 to D39, D3 to D4, D38 to D40, D40 to D41, D41 to D42, D42 to D43, D43 to D44, D44 to D45, D45 to D46, D46 to D47, D4 to D5, D5 to D6, D6 to D7, D7 to D8, D8 to D9, R6 to R1, R1 to R2, R2 to R3, R7 to R5, R5 to R6, R3 to R7, SW9 to SW10, SW10 to SW11, SW13 to SW16, SW14 to SW17, SW15 to SW18, SW16 to SW19, SW1 to SW2, SW17 to SW20, SW18 to SW21, SW19 to SW22, SW20 to SW23, SW21 to SW24, SW47 to SW27, SW24 to SW28, SW25 to SW29, SW2 to SW3, SW26 to SW30, SW27 to SW31, SW28 to SW32, SW29 to SW33, SW30 to SW34, SW31 to SW35, SW32 to SW36, SW35 to SW39, SW3 to SW4, SW38 to SW41, SW4 to SW5, SW5 to SW6, SW6 to SW7, SW7 to SW8, SW8 to SW9
Connections:
- SW43 pad 1: col7 -> col8
Routing:
- net Net-(D23-Pad2): track 0.00 -> 138.4 mm
- net Net-(D45-Pad2): track 149.1 -> 219.6 mm
- net Net-(D41-Pad2): track 98.5 -> 150.1 mm
- net Net-(D42-Pad2): track 125.2 -> 169.4 mm
- net col6: track 112.5 -> 144.2 mm
- net col8: track 77.9 -> 107.0 mm
- net col9: track 90.7 -> 116.9 mm
- net Net-(D11-Pad2): track 70.1 -> 45.9 mm
- net Net-(D44-Pad2): track 124.5 -> 146.7 mm
- net col1: track 203.1 -> 224.1 mm
- net Net-(D12-Pad2): track 96.3 -> 76.2 mm
- net col2: track 184.0 -> 203.4 mm
- net Net-(D43-Pad2): track 100.7 -> 119.7 mm
- net Net-(D33-Pad2): track 109.6 -> 128.0 mm
- net row1: track 332.3 -> 350.6 mm
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Other:
- rule pad_to_mask_clearance: 0.051 -> 0
- board text added: "1.25u"
- board text added: "1.5u"
- board text added: "1u"
- board text added: "2.25"
- board text added: "2.75"
- board text added: "2u back"
- board text added: "6.25"
- board text removed: "1.25U"
- board text removed: "1U"
- board text removed: "2.25U"
- board text removed: "2.75U"
- board text removed: "SPLIT"
- board text removed: "STANDARD"
- board text removed: "STEPPED"
