File: romeo-pcb.kicad_pcb (KiCad board)
At the start: 2 copper layers, 247.6 x 99.2 mm, 137 parts, among them J1 AVR-ISP-6, SW1 KEYSW, SW10 KEYSW, SW11 KEYSW, SW12 KEYSW, SW13 KEYSW, SW14 KEYSW, SW15 KEYSW, SW16 KEYSW, SW17 KEYSW, SW18 KEYSW, SW19 KEYSW, SW2 KEYSW, SW20 KEYSW, SW21 KEYSW, SW22 KEYSW, SW23 KEYSW, SW24 KEYSW, SW25 KEYSW, SW26 KEYSW, SW27 KEYSW, SW28 KEYSW, SW29 KEYSW, SW3 KEYSW, SW30 KEYSW, SW31 KEYSW, SW32 KEYSW, SW33 KEYSW, SW34 KEYSW, SW35 KEYSW, SW36 KEYSW, SW37 KEYSW, SW38 KEYSW, SW39 KEYSW, SW4 KEYSW, SW40 KEYSW, SW41 KEYSW, SW42 KEYSW, SW43 KEYSW, SW44 KEYSW, SW45 KEYSW, SW46 KEYSW, SW47 KEYSW, SW48 KEYSW, SW49 KEYSW, SW5 KEYSW, SW50 KEYSW, SW51 KEYSW, SW52 KEYSW, SW53 KEYSW, SW6 KEYSW, SW7 KEYSW, SW8 KEYSW, SW9 KEYSW, U1 ATmega328P-PU, Y1 Crystal

Commit message: Update silks and gerbers
Parts:
- added G***: LOGO, cc:cc, F.Cu at (201.6, 123.8)
- added Ref**: Val**, perso_silks:golmon_silk_svg, B.Cu at (50.6, 109.2)
- added Ref**: Val**, perso_silks:golmon_silk_svg, F.Cu at (242.9, 104.1)
- added Ref**: Val**, cftkb:putain_svg, F.Cu at (69.8, 49.2)
- added Ref**: Val**, cftkb:mkfr_footprint, B.Cu at (39.0, 123.8)
- added Ref**: Val**, cftkb:mkfr_footprint, F.Cu at (264.4, 121.6)
- added Ref**: Val**, cftkb:putain_svg, B.Cu at (234.2, 49.2)
