File: romeo-pcb.sch (KiCad schematic (older format))
At the start: 114 parts, among them J1 AVR-ISP-6, SW0 KEYSW, SW1 KEYSW, SW10 KEYSW, SW11 KEYSW, SW12 KEYSW, SW13 KEYSW, SW14 KEYSW, SW15 KEYSW, SW16 KEYSW, SW17 KEYSW, SW18 KEYSW, SW19 KEYSW, SW2 KEYSW, SW20 KEYSW, SW21 KEYSW, SW22 KEYSW, SW23 KEYSW, SW24 KEYSW, SW25 KEYSW, SW26 KEYSW, SW27 KEYSW, SW28 KEYSW, SW29 KEYSW, SW3 KEYSW, SW30 KEYSW, SW31 KEYSW, SW32 KEYSW, SW33 KEYSW, SW34 KEYSW, SW35 KEYSW, SW36 KEYSW, SW37 KEYSW, SW38 KEYSW, SW39 KEYSW, SW4 KEYSW, SW40 KEYSW, SW41 KEYSW, SW42 KEYSW, SW43 KEYSW, SW44 KEYSW, SW45 KEYSW, SW46 KEYSW, SW47 KEYSW, SW5 KEYSW, SW6 KEYSW, SW7 KEYSW, SW8 KEYSW, SW9 KEYSW, U1 ATmega328P-PU, Y1 Crystal

Commit message: Add new layout to romeo keyboard
Add the new layout (based on CC45) to make the keyboard more convenient to use
Update footprints to match this rev1.2
Parts:
- removed SW45, SW46: KEYSW, cftkb:SW_Cherry_MX1A_1.25u_PCBNOSCREEN, symbol keyboard_parts:KEYSW
- added D23: D_Small, cftkb:D_DO-35_SOD27_P5.08mm_Horizontal, symbol Device:D_Small
- added SW13: KEYSW, cftkb:SW_Cherry_MX1A_2.00u_PCBNOSCREEN, symbol romeo-pcb-rescue:KEYSW-keyboard_parts
- added SW14, SW49, SW52: KEYSW, cftkb:SW_Cherry_MX1A_1.00u_PCB-NOSCREEN, symbol romeo-pcb-rescue:KEYSW-keyboard_parts
- added SW48, SW50, SW51: KEYSW, cftkb:SW_Cherry_MX1A_1.25u_PCBNOSCREEN, symbol romeo-pcb-rescue:KEYSW-keyboard_parts
- SW1: renamed from SW0; footprint cftkb:SW_Cherry_MX1A_1.50u_PCBNOSCREEN -> cftkb:SW_Cherry_MX1A_1.00u_PCB-NOSCREEN; symbol keyboard_parts:KEYSW -> romeo-pcb-rescue:KEYSW-keyboard_parts
- SW10: renamed from SW9; symbol keyboard_parts:KEYSW -> romeo-pcb-rescue:KEYSW-keyboard_parts
- SW11: renamed from SW10; symbol keyboard_parts:KEYSW -> romeo-pcb-rescue:KEYSW-keyboard_parts
- SW12: renamed from SW11; footprint cftkb:SW_Cherry_MX1A_1.50u_PCBNOSCREEN -> cftkb:SW_Cherry_MX1A_1.00u_PCB-NOSCREEN; symbol keyboard_parts:KEYSW -> romeo-pcb-rescue:KEYSW-keyboard_parts
- SW15: renamed from SW12; footprint cftkb:SW_Cherry_MX1A_1.75u_PCBNOSCREEN -> cftkb:SW_Cherry_MX1A_1.25u_PCBNOSCREEN; symbol keyboard_parts:KEYSW -> romeo-pcb-rescue:KEYSW-keyboard_parts
- SW16: renamed from SW13; symbol keyboard_parts:KEYSW -> romeo-pcb-rescue:KEYSW-keyboard_parts
- SW17: renamed from SW14; symbol keyboard_parts:KEYSW -> romeo-pcb-rescue:KEYSW-keyboard_parts
- SW18: renamed from SW15; symbol keyboard_parts:KEYSW -> romeo-pcb-rescue:KEYSW-keyboard_parts
- SW19: renamed from SW16; symbol keyboard_parts:KEYSW -> romeo-pcb-rescue:KEYSW-keyboard_parts
- SW2: renamed from SW1; symbol keyboard_parts:KEYSW -> romeo-pcb-rescue:KEYSW-keyboard_parts
- SW20: renamed from SW17; symbol keyboard_parts:KEYSW -> romeo-pcb-rescue:KEYSW-keyboard_parts
- SW21: renamed from SW18; symbol keyboard_parts:KEYSW -> romeo-pcb-rescue:KEYSW-keyboard_parts
- SW22: renamed from SW19; symbol keyboard_parts:KEYSW -> romeo-pcb-rescue:KEYSW-keyboard_parts
- SW23: renamed from SW20; symbol keyboard_parts:KEYSW -> romeo-pcb-rescue:KEYSW-keyboard_parts
- SW24: renamed from SW21; symbol keyboard_parts:KEYSW -> romeo-pcb-rescue:KEYSW-keyboard_parts
- SW25: renamed from SW22; footprint cftkb:SW_Cherry_MX1A_2.25u_PCBNOSCREEN -> cftkb:SW_Cherry_MX1A_1.75u_PCBNOSCREEN; symbol keyboard_parts:KEYSW -> romeo-pcb-rescue:KEYSW-keyboard_parts
- SW26: renamed from SW23; footprint cftkb:SW_Cherry_MX1A_2.25u_PCBNOSCREEN -> cftkb:SW_Cherry_MX1A_1.75u_PCBNOSCREEN; symbol keyboard_parts:KEYSW -> romeo-pcb-rescue:KEYSW-keyboard_parts
- SW27: renamed from SW47; symbol keyboard_parts:KEYSW -> romeo-pcb-rescue:KEYSW-keyboard_parts
- SW28: renamed from SW24; symbol keyboard_parts:KEYSW -> romeo-pcb-rescue:KEYSW-keyboard_parts
- SW29: renamed from SW25; symbol keyboard_parts:KEYSW -> romeo-pcb-rescue:KEYSW-keyboard_parts
- SW3: renamed from SW2; symbol keyboard_parts:KEYSW -> romeo-pcb-rescue:KEYSW-keyboard_parts
- SW30: renamed from SW26; symbol keyboard_parts:KEYSW -> romeo-pcb-rescue:KEYSW-keyboard_parts
- SW31: renamed from SW27; symbol keyboard_parts:KEYSW -> romeo-pcb-rescue:KEYSW-keyboard_parts
- SW32: renamed from SW28; symbol keyboard_parts:KEYSW -> romeo-pcb-rescue:KEYSW-keyboard_parts
- SW33: renamed from SW29; symbol keyboard_parts:KEYSW -> romeo-pcb-rescue:KEYSW-keyboard_parts
- SW34: renamed from SW30; symbol keyboard_parts:KEYSW -> romeo-pcb-rescue:KEYSW-keyboard_parts
- SW35: renamed from SW31; symbol keyboard_parts:KEYSW -> romeo-pcb-rescue:KEYSW-keyboard_parts
- SW36: renamed from SW32; symbol keyboard_parts:KEYSW -> romeo-pcb-rescue:KEYSW-keyboard_parts
- SW37: renamed from SW33; footprint cftkb:SW_Cherry_MX1A_1.75u_PCBNOSCREEN -> cftkb:SW_Cherry_MX1A_1.25u_PCBNOSCREEN; symbol keyboard_parts:KEYSW -> romeo-pcb-rescue:KEYSW-keyboard_parts
- SW38: renamed from SW34; footprint cftkb:SW_Cherry_MX1A_1.25u_PCBNOSCREEN -> cftkb:SW_Cherry_MX1A_1.50u_PCBNOSCREEN; symbol keyboard_parts:KEYSW -> romeo-pcb-rescue:KEYSW-keyboard_parts
- SW39: renamed from SW35; symbol keyboard_parts:KEYSW -> romeo-pcb-rescue:KEYSW-keyboard_parts
- SW4: renamed from SW3; symbol keyboard_parts:KEYSW -> romeo-pcb-rescue:KEYSW-keyboard_parts
- SW40: renamed from SW36; footprint cftkb:SW_Cherry_MX1A_1.00u_PCB-NOSCREEN -> cftkb:SW_Cherry_MX1A_1.50u_PCBNOSCREEN; symbol keyboard_parts:KEYSW -> romeo-pcb-rescue:KEYSW-keyboard_parts
- SW41: renamed from SW38; symbol keyboard_parts:KEYSW -> romeo-pcb-rescue:KEYSW-keyboard_parts
- SW42: renamed from SW40; footprint cftkb:SW_Cherry_MX1A_1.00u_PCB-NOSCREEN -> MX_Only:MXOnly-2.75U-ReversedStabilizers-NoLED; symbol keyboard_parts:KEYSW -> romeo-pcb-rescue:KEYSW-keyboard_parts
- SW43: renamed from SW41; footprint cftkb:SW_Cherry_MX1A_2.75u_PCB_NOSCREEN -> cftkb:SW_Cherry_MX1A_1.50u_PCBNOSCREEN; symbol keyboard_parts:KEYSW -> romeo-pcb-rescue:KEYSW-keyboard_parts
- SW44: renamed from SW42; footprint cftkb:SW_Cherry_MX1A_1.25u_PCBNOSCREEN -> cftkb:SW_Cherry_MX1A_1.00u_PCB-NOSCREEN; symbol keyboard_parts:KEYSW -> romeo-pcb-rescue:KEYSW-keyboard_parts
- SW45: renamed from SW43; footprint cftkb:SW_Cherry_MX1A_1.00u_PCB-NOSCREEN -> cftkb:SW_Cherry_MX1A_1.50u_PCBNOSCREEN; symbol keyboard_parts:KEYSW -> romeo-pcb-rescue:KEYSW-keyboard_parts
- SW46: renamed from SW44; footprint cftkb:SW_Cherry_MX1A_1.25u_PCBNOSCREEN -> cftkb:SW_Cherry_MX1A_1.00u_PCB-NOSCREEN; symbol keyboard_parts:KEYSW -> romeo-pcb-rescue:KEYSW-keyboard_parts
- SW47: renamed from SW39; footprint cftkb:SW_Cherry_MX1A_1.00u_PCB-NOSCREEN -> MX_Only:MXOnly-6.25U-ReversedStabilizers-NoLED; symbol keyboard_parts:KEYSW -> romeo-pcb-rescue:KEYSW-keyboard_parts
- SW5: renamed from SW4; symbol keyboard_parts:KEYSW -> romeo-pcb-rescue:KEYSW-keyboard_parts
- SW53: renamed from SW37; footprint cftkb:SW_Cherry_MX1A_1.25u_PCBNOSCREEN -> cftkb:SW_Cherry_MX1A_1.00u_PCB-NOSCREEN; symbol keyboard_parts:KEYSW -> romeo-pcb-rescue:KEYSW-keyboard_parts
- SW6: renamed from SW5; symbol keyboard_parts:KEYSW -> romeo-pcb-rescue:KEYSW-keyboard_parts
- SW7: renamed from SW6; symbol keyboard_parts:KEYSW -> romeo-pcb-rescue:KEYSW-keyboard_parts
- SW8: renamed from SW7; symbol keyboard_parts:KEYSW -> romeo-pcb-rescue:KEYSW-keyboard_parts
- SW9: renamed from SW8; symbol keyboard_parts:KEYSW -> romeo-pcb-rescue:KEYSW-keyboard_parts
- USB1: symbol Type-C:USB_C_GCT_USB4085 -> romeo-pcb-rescue:USB_C_GCT_USB4085-Type-C
- renumbered C3 to C1, C4 to C2, C5 to C3, C1 to C4, C2 to C5, D0 to D1, D9 to D10, D10 to D11, D11 to D12, D12 to D13, D13 to D14, D14 to D15, D15 to D16, D16 to D17, D17 to D18, D18 to D19, D1 to D2, D19 to D20, D20 to D21, D21 to D22, D22 to D24, D23 to D25, D47 to D26, D24 to D27, D25 to D28, D26 to D29, D2 to D3, D27 to D30, D28 to D31, D29 to D32, D30 to D33, D31 to D34, D32 to D35, D33 to D36, D34 to D37, D35 to D38, D36 to D39, D3 to D4, D38 to D40, D40 to D41, D41 to D42, D42 to D43, D43 to D44, D44 to D45, D45 to D46, D46 to D47, D4 to D5, D5 to D6, D6 to D7, D7 to D8, D8 to D9, R6 to R1, R1 to R2, R2 to R3, R7 to R5, R5 to R6, R3 to R7
Connections:
- wire segments 200 -> 221
Other:
- moved on the sheet: D42
