File: bottom/romeo-bottom.kicad_pcb (KiCad board)
At the start: 2 copper layers, 247.7 x 99.2 mm, 14 parts

Commit message: Update silks and gerbers
Parts:
- added REF**: putain_big_oval, cftkb:putain_big_oval, F.Cu at (145.1, 62.3)
Other:
- rule pad_to_mask_clearance: 0.051 -> 0

Commit message: Update gerbers, sent a first command to jlcpcb
Other:
- board text added: "JLCJLCJLCJLC"
Changed lines of the file:
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@@
-(kicad_pcb (version 20171130) (host pcbnew "(5.1.9)-1")
+(kicad_pcb (version 20171130) (host pcbnew "(5.1.10)-1")
   (general
     (thickness 1.6)
-    (drawings 10)
+    (drawings 11)
     (tracks 0)
     (zones 0)
@@
     (pad 1 thru_hole circle (at 0 0) (size 4.4 4.4) (drill 2.2) (layers *.Cu *.Mask))
   )
+  (gr_text JLCJLCJLCJLC (at 55 92) (layer B.SilkS)
+    (effects (font (size 1 1) (thickness 0.15)) (justify mirror))
+  )
   (gr_text coseyfannitutti (at 81.5848 76.5556) (layer B.Mask)
