File: plate/switch_plate/switch_plate.kicad_pcb (KiCad board)
At the start: 2 copper layers, 247.7 x 76.2 mm, 2 parts

Commit message: Update silks and gerbers
Routing:
- net (no net): vias 0 -> 1
Changed lines of the file:
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@@
     (thickness 1.6)
     (drawings 435)
-    (tracks 0)
+    (tracks 1)
     (zones 0)
     (modules 2)
@@
     (pad_to_mask_clearance 0)
     (aux_axis_origin 0 0)
-    (visible_elements FFFFFF7F)
+    (visible_elements 7FFFFFFF)
     (pcbplotparams
-      (layerselection 0x010fc_ffffffff)
+      (layerselection 0x010f0_ffffffff)
       (usegerberextensions false)
       (usegerberattributes true)
@@
       (outputformat 1)
       (mirror false)
-      (drillshape 1)
+      (drillshape 0)
       (scaleselection 1)
-      (outputdirectory ""))
+      (outputdirectory "../../Gerber/plate/"))
   )
   (net 0 "")
@@
   (gr_arc (start 146.2875 106.122949) (end 145.7875 106.122949) (angle -90) (layer Edge.Cuts) (width 0.2))
   (gr_arc (start 159.2875 93.122949) (end 159.7875 93.122949) (angle -90) (layer Edge.Cuts) (width 0.2))
+  (via (at 55.875 115) (size 0.8) (drill 0.4) (layers F.Cu B.Cu) (net 0))
   (zone (net 0) (net_name "") (layer F.Cu) (hatch edge 0.508)
     (connect_pads (clearance 0.508))

Commit message: Update gerbers, sent a first command to jlcpcb
Other:
- board text added: "JLCJLCJLCJLC"
Changed lines of the file:
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@@
-(kicad_pcb (version 20171130) (host pcbnew "(5.1.9)-1")
+(kicad_pcb (version 20171130) (host pcbnew "(5.1.10)-1")
   (general
     (thickness 1.6)
-    (drawings 435)
+    (drawings 436)
     (tracks 1)
     (zones 0)
@@
       (xy -2.227987 2.915569) (xy -2.172257 2.912252)) (layer B.Mask) (width 0.01))
   )
+  (gr_text JLCJLCJLCJLC (at 229.2 107.8) (layer B.SilkS)
+    (effects (font (size 1 1) (thickness 0.15)) (justify mirror))
+  )
   (gr_arc (start 91.65 130.22) (end 91.65 130.72) (angle -90) (layer Edge.Cuts) (width 0.2))
